File: PC104_ISA_8bits.kicad_sch (KiCad schematic)
At the start: 9 parts

Commit message: Fin de l'init
git-svn-id: file:///D%5C00%20-%20Dev%20&%20Calculs%5CRepoTortoiseSVN_PCB%5CPC104_Template/branches/PC104_ISA_8bits@11 5901225d-b6fc-0a46-af7b-916857fbd23b
Parts:
- Bus_ISA_8bit_1: footprint Connector_PinSocket_2.54mm:PinSocket_2x32_P2.54mm_Vertical -> Conn_ISA_8bits:PinSocket_2x32_P2.54mm_Vertical_TopBottom
Changed lines of the file:
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@@
   (symbol (lib_id "power:+5V") (at 142.24 49.53 90) (unit 1)
     (in_bom yes) (on_board yes) (dnp no)
-    (property "Reference" "#PWR0108" (at 146.05 49.53 0)
+    (property "Reference" "#PWR?" (at 146.05 49.53 0)
       (effects (font (size 1.27 1.27)) hide)
     )
@@
       (project "PC104_ISA_8bits"
         (path "/b26d10c1-0874-459a-80a4-e525262e670c"
-          (reference "#PWR0108") (unit 1)
+          (reference "#PWR?") (unit 1)
         )
       )
@@
       (effects (font (size 1.27 1.27)))
     )
-    (property "Footprint" "Connector_PinSocket_2.54mm:PinSocket_2x32_P2.54mm_Vertical" (at 172.72 130.81 0)
+    (property "Footprint" "Conn_ISA_8bits:PinSocket_2x32_P2.54mm_Vertical_TopBottom" (at 172.72 130.81 0)
       (effects (font (size 1.27 1.27)) hide)
     )
@@
   (symbol (lib_id "power:+5V") (at 142.24 115.57 90) (unit 1)
     (in_bom yes) (on_board yes) (dnp no)
-    (property "Reference" "#PWR0113" (at 146.05 115.57 0)
+    (property "Reference" "#PWR?" (at 146.05 115.57 0)
       (effects (font (size 1.27 1.27)) hide)
     )
@@
       (project "PC104_ISA_8bits"
         (path "/b26d10c1-0874-459a-80a4-e525262e670c"
-          (reference "#PWR0113") (unit 1)
+          (reference "#PWR?") (unit 1)
         )
       )
@@
   (symbol (lib_id "power:GND") (at 148.59 120.65 0) (unit 1)
     (in_bom yes) (on_board yes) (dnp no)
-    (property "Reference" "#PWR0112" (at 148.59 127 0)
+    (property "Reference" "#PWR?" (at 148.59 127 0)
       (effects (font (size 1.27 1.27)) hide)
     )
@@
       (project "PC104_ISA_8bits"
         (path "/b26d10c1-0874-459a-80a4-e525262e670c"
-          (reference "#PWR0112") (unit 1)
+          (reference "#PWR?") (unit 1)
         )
       )
@@
   (symbol (lib_id "power:GND") (at 148.59 41.91 180) (unit 1)
     (in_bom yes) (on_board yes) (dnp no)
-    (property "Reference" "#PWR0103" (at 148.59 35.56 0)
+    (property "Reference" "#PWR?" (at 148.59 35.56 0)
       (effects (font (size 1.27 1.27)) hide)
     )
@@
       (project "PC104_ISA_8bits"
         (path "/b26d10c1-0874-459a-80a4-e525262e670c"
-          (reference "#PWR0103") (unit 1)
+          (reference "#PWR?") (unit 1)
         )
       )
@@
   (symbol (lib_id "power:GND") (at 194.31 41.91 180) (unit 1)
     (in_bom yes) (on_board yes) (dnp no)
-    (property "Reference" "#PWR0107" (at 194.31 35.56 0)
+    (property "Reference" "#PWR?" (at 194.31 35.56 0)
       (effects (font (size 1.27 1.27)) hide)
     )
@@
       (project "PC104_ISA_8bits"
         (path "/b26d10c1-0874-459a-80a4-e525262e670c"
-          (reference "#PWR0107") (unit 1)
-        )
-      )
+          (reference "#PWR?") (unit 1)
+        )
+      )

Commit message: git-svn-id: file:///D%5C00%20-%20Dev%20&%20Calculs%5CRepoTortoiseSVN_PCB%5CPC104_Template/branches/PC104_ISA_8bits@9 5901225d-b6fc-0a46-af7b-916857fbd23b
Parts:
- Bus_ISA_8bit_1: footprint Conn_ISA_8bits:PinSocket_2x32_P2.54mm_Vertical_TopBottom -> Connector_PinSocket_2.54mm:PinSocket_2x32_P2.54mm_Vertical
Changed lines of the file:
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@@
   (symbol (lib_id "power:+5V") (at 142.24 49.53 90) (unit 1)
     (in_bom yes) (on_board yes) (dnp no)
-    (property "Reference" "#PWR?" (at 146.05 49.53 0)
+    (property "Reference" "#PWR0108" (at 146.05 49.53 0)
       (effects (font (size 1.27 1.27)) hide)
     )
@@
       (project "PC104_ISA_8bits"
         (path "/b26d10c1-0874-459a-80a4-e525262e670c"
-          (reference "#PWR?") (unit 1)
+          (reference "#PWR0108") (unit 1)
         )
       )
@@
       (effects (font (size 1.27 1.27)))
     )
-    (property "Footprint" "Conn_ISA_8bits:PinSocket_2x32_P2.54mm_Vertical_TopBottom" (at 172.72 130.81 0)
+    (property "Footprint" "Connector_PinSocket_2.54mm:PinSocket_2x32_P2.54mm_Vertical" (at 172.72 130.81 0)
       (effects (font (size 1.27 1.27)) hide)
     )
@@
   (symbol (lib_id "power:+5V") (at 142.24 115.57 90) (unit 1)
     (in_bom yes) (on_board yes) (dnp no)
-    (property "Reference" "#PWR?" (at 146.05 115.57 0)
+    (property "Reference" "#PWR0113" (at 146.05 115.57 0)
       (effects (font (size 1.27 1.27)) hide)
     )
@@
       (project "PC104_ISA_8bits"
         (path "/b26d10c1-0874-459a-80a4-e525262e670c"
-          (reference "#PWR?") (unit 1)
+          (reference "#PWR0113") (unit 1)
         )
       )
@@
   (symbol (lib_id "power:GND") (at 148.59 120.65 0) (unit 1)
     (in_bom yes) (on_board yes) (dnp no)
-    (property "Reference" "#PWR?" (at 148.59 127 0)
+    (property "Reference" "#PWR0112" (at 148.59 127 0)
       (effects (font (size 1.27 1.27)) hide)
     )
@@
       (project "PC104_ISA_8bits"
         (path "/b26d10c1-0874-459a-80a4-e525262e670c"
-          (reference "#PWR?") (unit 1)
+          (reference "#PWR0112") (unit 1)
         )
       )
@@
   (symbol (lib_id "power:GND") (at 148.59 41.91 180) (unit 1)
     (in_bom yes) (on_board yes) (dnp no)
-    (property "Reference" "#PWR?" (at 148.59 35.56 0)
+    (property "Reference" "#PWR0103" (at 148.59 35.56 0)
       (effects (font (size 1.27 1.27)) hide)
     )
@@
       (project "PC104_ISA_8bits"
         (path "/b26d10c1-0874-459a-80a4-e525262e670c"
-          (reference "#PWR?") (unit 1)
+          (reference "#PWR0103") (unit 1)
         )
       )
@@
   (symbol (lib_id "power:GND") (at 194.31 41.91 180) (unit 1)
     (in_bom yes) (on_board yes) (dnp no)
-    (property "Reference" "#PWR?" (at 194.31 35.56 0)
+    (property "Reference" "#PWR0107" (at 194.31 35.56 0)
       (effects (font (size 1.27 1.27)) hide)
     )
@@
       (project "PC104_ISA_8bits"
         (path "/b26d10c1-0874-459a-80a4-e525262e670c"
-          (reference "#PWR?") (unit 1)
-        )
-      )
+          (reference "#PWR0107") (unit 1)
+        )
+      )
