File: PC104_PCI_CAN_Express/Connection PCI CAN Express.kicad_sch (KiCad schematic)
At the start: 1 part, among them J1 Conn_02x20_Odd_Even

Commit message: UPDATE : Connecteur unique avec trous NPTH
Connections:
- no-connect marks 0 -> 4
Changed lines of the file:
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@@
 (kicad_sch
-	(version 20250114)
+	(version 20260306)
 	(generator "eeschema")
-	(generator_version "9.0")
+	(generator_version "10.0")
 	(paper "A4")
 	(text "Liaison :\n	- PRSNT1# et PRSNT2# par le GNDD (équivalent présence carte PCIx1)\n\nRemplacement :\n	- SMBus -> I2C\n	- JTAG -> SPI dont SC1# et SC2#\n	- WAKE# -> CS3#\n	- CLKREQ -> CLKO\n	- RefClk différentielle PCI -> OSC1 et OSC2 pour external clock MCU\n	- HSOp(0) soit TX0 PCI -> ModBus A+\n	- HSOn(0) soit TX0 PCI -> ModBus B-\n	- HSIp(0) soit RXO PCI -> CAN_0_H\n	- HSIn(0) soit RXO PCI -> CAN_0_L\n\nPS : \nL'utilisation d'un RS485 4 fils est possibles en cablant :\n	- HSOp(0) soit TX0 PCI -> DI_A+ master / RO_A+ slave(s)\n	- HSOn(0) soit TX0 PCI -> DI_B- master / RO_B- slave(s)\n	- HSIp(0) soit RXO PCI -> RO_A+ master / DI_A+ slave(s)\n	- HSIn(0) soit RXO PCI -> RO_B- master / DI_B- slave(s)\n\nL'utilisation d'un RS485 2 fils est possibles en cablant :\n	- HSOp(0) soit TX0 PCI -> A+ master / A+ slave\n	- HSOn(0) soit TX0 PCI -> B- master / B- slave\n	- HSIp(0) soit RXO PCI -> NC. ou CAN_0_H\n	- HSIn(0) soit RXO PCI -> NC. ou CAN_0_L\n"
@@
 		)
 	)
+	(no_connect
+		(at 78.74 101.6)
+	)
+	(no_connect
+		(at 91.44 101.6)
+	)
+	(no_connect
+		(at 91.44 99.06)
+	)
+	(no_connect
+		(at 78.74 99.06)
+	)
 	(wire
 		(pts
@@
 		(at 83.82 93.98 0)
 		(unit 1)
+		(body_style 1)
 		(exclude_from_sim no)
 		(in_bom yes)
 		(on_board yes)
+		(in_pos_files yes)
 		(dnp no)
 		(fields_autoplaced yes)
 		(property "Reference" "J1"
 			(at 85.09 64.77 0)
+			(show_name no)
+			(do_not_autoplace no)
 			(effects
 				(font
@@
 		(property "Value" "Conn_02x20_Odd_Even"
 			(at 85.09 67.31 0)
+			(show_name no)
+			(do_not_autoplace no)
 			(effects
 				(font
@@
 		(property "Footprint" "Connector_IDC:IDC-Header_2x20_P2.54mm_Vertical"
 			(at 83.82 93.98 0)
+			(hide yes)
+			(show_name no)
+			(do_not_autoplace no)
 			(effects
 				(font
 					(size 1.27 1.27)
 				)
-				(hide yes)
 			)
 		)
-		(property "Datasheet" "~"
+		(property "Datasheet" ""
 			(at 83.82 93.98 0)
+			(hide yes)
+			(show_name no)
+			(do_not_autoplace no)
 			(effects
 				(font
 					(size 1.27 1.27)
 				)
-				(hide yes)
 			)
 		)
 		(property "Description" "Generic connector, double row, 02x20, odd/even pin numbering scheme (row 1 odd numbers, row 2 even numbers), script generated (kicad-library-utils/schlib/autogen/connector/)"
 			(at 83.82 93.98 0)
+			(hide yes)
+			(show_name no)
+			(do_not_autoplace no)
 			(effects
 				(font
 					(size 1.27 1.27)
 				)
-				(hide yes)
 			)
 		)
@@
 		)
 		(instances
-			(project ""
+			(project "PC104_PCI_CAN_Express"
 				(path "/b26d10c1-0874-459a-80a4-e525262e670c/49081260-d3db-4891-bc97-e468d504baf8"
 					(reference "J1")
